File: pcb/ignition/ignition.kicad_pcb (KiCad board)
At the start: 4 copper layers, 100 x 100 mm, 146 parts, among them IC1 LTC4151, IC2 LTC4151, IC3 LTC4151, IC4 LTC4151, IC5 LTC4151, IC6 LTC4151, IC7 ADP3335, IC8 STM32F437VIT6, J1 PSU, J10 CH2, J11 CH4, J12 ARM, J13 UART1, J14 UART2, J15 CH1, J16 CH3, J17 CH5, J2 LED1, J3 PSU, J4 LED2, J5 5v In, J6 5v Out, J7 LED3, J8 LED4, J9 LED5, K1 16A SPST, K2 16A SPST, K3 16A SPST, K4 16A SPST, K5 16A SPST, K6 16A SPST, P1 SWD_TC, Q1 NFET, Q2 NFET, Q3 NFET, Q4 NFET, Q5 NFET, Q6 NFET, U1 MICROSD, X33 Hole, X34 Hole, X35 Hole, X36 Hole, Y1 26M

Commit message: production ready gerbers for ignition
Other:
- rule solder_mask_min_width: 0.25 -> 0.1
Changed lines of the file:
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@@
     (pad_drill 3.048)
     (pad_to_mask_clearance 0)
-    (solder_mask_min_width 0.25)
+    (solder_mask_min_width 0.1)
     (aux_axis_origin 0 0)
     (visible_elements FFFFFF5F)
@@
       (plotinvisibletext false)
       (padsonsilk false)
-      (subtractmaskfromsilk true)
+      (subtractmaskfromsilk false)
       (outputformat 1)
       (mirror false)
