File: pcb/ignition/ignition.sch (KiCad schematic (older format))
At the start: 178 parts, among them IC1 LTC4151, IC2 LTC4151, IC3 LTC4151, IC4 LTC4151, IC5 LTC4151, IC6 LTC4151, IC7 ADP3335, IC8 STM32F437VIT6, J1 PSU, J10 CH2, J11 CH4, J12 ARM, J13 UART1, J14 UART2, J15 CH1, J16 CH3, J17 CH5, J2 LED1, J3 PSU, J4 LED2, J5 5v In, J6 5v Out, J7 LED3, J8 LED4, J9 LED5, K1 16A SPST, K2 16A SPST, K3 16A SPST, K4 16A SPST, K5 16A SPST, K6 16A SPST, P1 SWD_TC, Q1 NFET, Q2 NFET, Q3 NFET, Q4 NFET, Q5 NFET, Q6 NFET, U1 MICROSD, X1 Molex Wire, X10 GRN LED, X11 LED Bezel, X12 24V PSU, X13 5V PSU, X14 GRN LED, X15 LED Bezel, X16 Molex Wire, X17 M12 Socket, X18 M12 Plug, X19 Molex Wire, X2 GRN LED, X20 M12 Socket, X21 M12 Plug, X22 Bi-LED, X23 LED Bezel, X24 Molex Wire, X25 M12 Socket, X26 M12 Plug, X27 Molex Wire, X28 M12 Socket, X29 M12 Plug, X3 LED Bezel, X30 Molex Wire, X31 M12 Socket, X32 M12 Plug, X33 Hole, X34 Hole, X35 Hole, X36 Hole, X4 GRN LED, X5 LED Bezel, X6 GRN LED, X7 LED Bezel, X8 Key Switch, X9 AC Input, Y1 26M

Commit message: added Boms
Parts:
- J10: Farnell 172316-1104 -> 2494369
Changed lines of the file:
@@
 F 2 "ignition:172316-1104" H 4900 5175 50  0001 C CNN
 F 3 "https://www.molex.com/pdm_docs/sd/1723161104_sd.pdf" H 4900 5175 50  0001 C CNN
-F 4 "172316-1104" H 4900 5175 50  0001 C CNN "Farnell"
+F 4 "2494369" H 4900 5175 50  0001 C CNN "Farnell"
 	1    4900 5175
 	-1   0    0    -1
