File: pcb/comms/comms.kicad_pcb (KiCad board)
At the start: 4 copper layers, 80 x 50 mm, 50 parts, among them IC1 STM32F437VIT6, IC2 ADP3335, IC3 MAX14787E, IC4 RJHSE-538x, J1 UART1, J2 UART2, J3 5v In, P1 USB-B, P2 SWD_TC, X5 Hole, X6 Hole, X8 Hole, X9 Hole, Y1 26M

Commit message: production ready gerbers
Other:
- rule solder_mask_min_width: 0.25 -> 0.1
Changed lines of the file:
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@@
     (pad_drill 0.762)
     (pad_to_mask_clearance 0)
-    (solder_mask_min_width 0.25)
+    (solder_mask_min_width 0.1)
     (aux_axis_origin 0 0)
     (visible_elements FFFFFF5F)
@@
       (plotinvisibletext false)
       (padsonsilk false)
-      (subtractmaskfromsilk true)
+      (subtractmaskfromsilk false)
       (outputformat 1)
       (mirror false)
